Commit message: mobile robot base urdf done

File: src/warehouse_robot_description/urdf/mobile_base.urdf.xacro (robot description, xacro)
@@ -1,17 +1,14 @@
 <?xml version="1.0"?>
 <robot xmlns:xacro="http://www.ros.org/wiki/xacro" name="warehouse_robot">
-    <!--==================================-->
-    <!--   DEFINE PROPERTIES (VARIABLES)-->
-    <!--=================================-->
-    <!-- Robot Dimensions(meters) -->
-    <xacro:property name="base_width" value="0.4"/> <!--40 cm wide-->
-    <xacro:property name="base_length" value="0.6"/> <!--60 cm long-->
-    <xacro:property name="base_height" value="0.2"/> <!--20 cm tall-->
-    <!-- Wheel Dimensions-->
-    <xacro:property name="wheel_radius" value="0.1"/> <!--10 cm radius-->
-    <xacro:property name="wheel_width" value="0.05"/> <!-- 5 cm wide-->
-    <xacro:property name="wheel_mass" value="0.5"/> <!--500 grams-->
-    <xacro:property name="base_mass" value="5.0"/>
-    <!-- MATERIALS (COLORS) -->
+    <!--Robot Base Properties (Variables) -->
+    <xacro:property name="base_length" value="0.6"/>
+    <xacro:property name="base_width" value="0.4"/>
+    <xacro:property name="base_height" value="0.2"/>
+    <xacro:property name="base_mass" value="10.0"/>
+    <xacro:property name="wheel_radius" value="0.1"/>
+    <xacro:property name="wheel_length" value="0.05"/>
+    <xacro:property name="wheel_mass" value="0.5"/>
+    <xacro:property name="caster_radius" value="0.05"/>
+    <xacro:property name="caster_mass" value="1.0"/>
     <material name="blue">
         <color rgba="0.2 0.2 0.8 1.0"/>
@@ -26,15 +23,18 @@
         <color rgba="0.9 0.9 0.9 1.0"/>
     </material>
-    <!-- ====== LINKS ======== -->
+    <!-- ============================== -->
+    <!--          LINKS                 -->
+    <!-- ============================== -->
+    <!-- Base Link -->
     <link name="base_link">
         <visual>
-            <origin xyz="0 0 ${base_height/2}" rpy="0 0 0"/>
+            <origin xyz="0 0 0" rpy="0 0 0"/>
             <geometry>
-                <box size="${base_length} ${base_width} ${base_height}"/>
+                <box size= "${base_length} ${base_width} ${base_height}"/>
             </geometry>
-            <material name="gray" />
+            <material name="blue"/>
         </visual>
         <collision>
-            <origin xyz="0 0 ${base_height/2}" rpy="0 0 0"/>
+            <origin xyz = "0 0 0" rpy = "0 0 0"/>
             <geometry>
                 <box size="${base_length} ${base_width} ${base_height}"/>
@@ -42,87 +42,95 @@
         </collision>
         <inertial>
-            <origin xyz="0 0 ${base_height/2}" rpy="0 0 0"/>
-            <mass value="${base_mass}"/>
-            <inertia ixx="0.1" iyy="0.1" izz="0.1"
+            <mass value="${base_mass}" />
+            <inertia ixx="0.1" iyy="0.33" izz="0.43"
                     ixy="0.0" ixz="0.0" iyz="0.0"/>
         </inertial>
     </link>
-    <!-- WHEEL MACRO AND LINK -->
-    <xacro:macro name="wheel_link" params="name x y z">
-        <link name="${name}">
-            <visual>
-            <origin xyz="${x} ${y} ${z}" rpy="1.5708 0 0"/>
+    <!-- Right Wheel -->
+    <link name="right_wheel">
+        <visual>
+            <origin xyz="0 0 0" rpy="1.57 0 0"/>
             <geometry>
-                <cylinder length="${wheel_width}" radius="${wheel_radius}"/>
+                <cylinder radius="${wheel_radius}" length="${wheel_length}"/>
             </geometry>
             <material name="black"/>
-            </visual>
-            <collision>
-            <origin xyz="${x} ${y} ${z}" rpy="1.5708 0 0"/>
+        </visual>
+        <collision>
+            <origin xyz="0 0 0" rpy="1.57 0 0"/>
             <geometry>
-                <cylinder length="${wheel_width}" radius="${wheel_radius}"/>
+                <cylinder radius="${wheel_radius}" length="${wheel_length}"/>
             </geometry>
-            </collision>
-            <inertial>
-            <origin xyz="${x} ${y} ${z}" rpy="1.5708 0 0"/>
+        </collision>
+        <inertial>
             <mass value="${wheel_mass}"/>
-            <inertia ixx="0.01" iyy="0.01" izz="0.01"
-                    ixy="0.0" ixz="0.0" iyz="0.0"/>
-            </inertial>
-        </link>
-    </xacro:macro>
-    <!-- ======================= -->
-    <!--   WHEEL LINKS PLACED    -->
-    <!-- ======================= -->
-    <!-- Front Left Wheel -->
-    <xacro:wheel_link name="wheel_front_left"
-                    x="${base_length/2 - wheel_width/2}"
-                    y="${base_width/2 - wheel_radius}"
-                    z="${wheel_radius}"/>
-    <!-- Front Right Wheel -->
-    <xacro:wheel_link name="wheel_front_right"
-                    x="${base_length/2 - wheel_width/2}"
-                    y="${-base_width/2 + wheel_radius}"
-                    z="${wheel_radius}"/>
-    <!-- Rear Left Wheel -->
-    <xacro:wheel_link name="wheel_rear_left"
-                    x="${-base_length/2 + wheel_width/2}"
-                    y="${base_width/2 - wheel_radius}"
-                    z="${wheel_radius}"/>
-    <!-- Rear Right Wheel -->
-    <xacro:wheel_link name="wheel_rear_right"
-                    x="${-base_length/2 + wheel_width/2}"
-                    y="${-base_width/2 + wheel_radius}"
-                    z="${wheel_radius}"/>
-    <!-- ======================= -->
-    <!--   JOINTS: WHEELS        -->
-    <!-- ======================= -->
-    <!-- Front Left -->
-    <joint name="joint_front_left_wheel" type="continuous">
-    <parent link="base_link"/>
-    <child link="wheel_front_left"/>
-    <origin xyz="${base_length/2 - wheel_width/2} ${base_width/2 - wheel_radius} ${wheel_radius}" rpy="0 0 0"/>
-    <axis xyz="0 1 0"/>
+            <inertia ixx="0.1" iyy="0.1" izz="0.1"
+                ixy="0.0" ixz="0.0" iyz="0.0"/>
+        </inertial>
+    </link>
+    <!-- Left Wheel-->
+    <link name="left_wheel">
+        <visual>
+            <origin xyz="0 0 0" rpy="1.57 0 0"/>
+            <geometry>
+                <cylinder radius="${wheel_radius}" length="${wheel_length}"/>
+            </geometry>
+            <material name="black"/>
+        </visual>
+        <collision>
+            <origin xyz="0 0 0" rpy="1.57 0 0"/>
+            <geometry>
+                <cylinder radius="${wheel_radius}" length="${wheel_length}"/>
+            </geometry>
+        </collision>
+        <inertial>
+            <mass value="${wheel_mass}"/>
+            <inertia ixx="0.1" iyy="0.1" izz="0.1"
+                ixy="0.0" ixz="0.0" iyz="0.0"/>
+        </inertial>
+    </link>
+    <!-- Caster Wheel -->
+    <link name="caster_wheel">
+        <visual>
+            <origin xyz="0 0 0" rpy="1.57 0 0"/>
+            <geometry>
+                <sphere radius="${caster_radius}"/>
+            </geometry>
+            <material name="white"/>
+        </visual>
+        <collision>
+            <origin xyz="0 0 0" rpy="1.57 0 0"/>
+            <geometry>
+                <sphere radius="${caster_radius}"/>
+            </geometry>
+        </collision>
+        <inertial>
+            <mass value="${caster_mass}"/>
+            <inertia ixx="0.1" iyy="0.1" izz="0.1"
+                ixy="0.0" ixz="0.0" iyz="0.0"/>
+        </inertial>
+    </link>
+    <!-- ============================== -->
+    <!--          JOINTS                -->
+    <!-- ============================== -->
+    <!-- right to base wheel -->
+    <joint name="right_wheel_to_base" type="continuous">
+        <parent link="base_link"/>
+        <child link="right_wheel"/>
+        <origin xyz="0 -0.225 -${wheel_radius}" rpy="0 0 0"/>
+        <axis xyz="0 1 0"/>
     </joint>
-    <!-- Front Right -->
-    <joint name="joint_front_right_wheel" type="continuous">
-    <parent link="base_link"/>
-    <child link="wheel_front_right"/>
-    <origin xyz="${base_length/2 - wheel_width/2} ${-base_width/2 + wheel_radius} ${wheel_radius}" rpy="0 0 0"/>
-    <axis xyz="0 1 0"/>
+    <!-- left wheel to base  -->
+    <joint name="left_wheel_to_base" type="continuous">
+        <parent link="base_link"/>
+        <child link="left_wheel"/>
+        <origin xyz="0 0.225 -${wheel_radius}" rpy="0 0 0"/>
+        <axis xyz="0 1 0"/>
     </joint>
-    <!-- Rear Left -->
-    <joint name="joint_rear_left_wheel" type="continuous">
-    <parent link="base_link"/>
-    <child link="wheel_rear_left"/>
-    <origin xyz="${-base_length/2 + wheel_width/2} ${base_width/2 - wheel_radius} ${wheel_radius}" rpy="0 0 0"/>
-    <axis xyz="0 1 0"/>
-    </joint>
-    <!-- Rear Right -->
-    <joint name="joint_rear_right_wheel" type="continuous">
-    <parent link="base_link"/>
-    <child link="wheel_rear_right"/>
-    <origin xyz="${-base_length/2 + wheel_width/2} ${-base_width/2 + wheel_radius} ${wheel_radius}" rpy="0 0 0"/>
-    <axis xyz="0 1 0"/>
+    <!-- Caster Wheel to base-->
+    <joint name="caster_wheel_to_base" type="fixed">
+        <parent link="base_link"/>
+        <child link="caster_wheel"/>
+        <origin xyz="0.25 0 -0.15" rpy="0 0 0"/>
+        <axis xyz="0 1 0"/>
     </joint>
 </robot>
