Commit message: URDF and Gazebo world done

File: src/warehouse_robot_description/urdf/gripper.urdf.xacro (robot description, xacro)
@@ -1 +1,125 @@
 <?xml version="1.0"?>
+<robot xmlns:xacro="http://www.ros.org/wiki/xacro">
+    <!-- 6 DOF MANIPULATOR MODULE
+    6. Degrees of Freedom
+    1. Base Rotation(yaw)
+    2. Shoulder pitch
+    3. shoulder roll
+    4. elbow pitch
+    5. wrist pitch
+    6. writch roll
+     + 2 DOF gripper (fingers) -->
+    <!-- LINK DIMENSIONS -->
+    <!-- Link6 - Shoulder Pitch -->
+    <xacro:property name="link6_length" value="0.04"/>
+    <!-- Gripper Dimensions  -->
+    <xacro:property name="gripper_base_length" value="0.05"/>
+    <xacro:property name="gripper_base_width" value="0.04"/>
+    <xacro:property name="gripper_base_height" value="0.03"/>
+    <xacro:property name="gripper_base_mass" value="0.1"/>
+    <xacro:property name="finger_length" value="0.08"/>
+    <xacro:property name="finger_width" value="0.015"/>
+    <xacro:property name="finger_height" value="0.025"/>
+    <xacro:property name="finger_mass" value="0.05"/>
+    <!-- INERTIA MACRO -->
+    <!-- Box inertia for Gripper Part-->
+    <xacro:macro name="box_inertia" params="mass x y z">
+        <inertia ixx = "${mass * (y*y + z*z)/12}"
+                iyy = "${mass * (x*x + z*z)/12}"
+                izz = "${mass * (x*x +y*y)/12}"
+                iyz = "0.0"
+                ixz = "0.0"
+                ixy = "0.0" />
+    </xacro:macro>
+    <!-- Main Manipulator Links Macro -->
+    <xacro:macro name="gripper" params="parent">
+        <!-- GRIPPER BASE -->
+      <link name="gripper_base">
+        <visual>
+          <origin xyz="0 0 ${gripper_base_length/2}" rpy="0 0 0"/>
+          <geometry>
+            <box size="${gripper_base_length} ${gripper_base_width} ${gripper_base_height}"/>
+          </geometry>
+          <material name="grey1"/>
+        </visual>
+        <collision>
+          <origin xyz="0 0 ${gripper_base_length/2}" rpy="0 0 0"/>
+          <geometry>
+            <box size="${gripper_base_length} ${gripper_base_width} ${gripper_base_height}"/>
+          </geometry>
+        </collision>
+        <inertial>
+          <mass value="${gripper_base_mass}"/>
+          <xacro:box_inertia mass="${gripper_base_mass}" x="${gripper_base_length}" y="${gripper_base_width}" z="${gripper_base_height}"/>
+          <origin xyz="0 0 ${gripper_base_length/2}" rpy = "0 0 0"/>
+        </inertial>
+      </link>
+        <!-- LEFT FINGER -->
+      <link name="left_finger">
+        <visual>
+          <origin xyz="0 0 ${finger_length/2}" rpy="0 0 0"/>
+          <geometry>
+            <box size="${finger_length} ${finger_width} ${finger_height}"/>
+          </geometry>
+          <material name="grey1"/>
+        </visual>
+        <collision>
+          <origin xyz="0 0 ${finger_length/2}" rpy="0 0 0"/>
+          <geometry>
+              <box size="${finger_length} ${finger_width} ${finger_height}"/>
+          </geometry>
+        </collision>
+        <inertial>
+          <mass value="${finger_mass}"/>
+          <xacro:box_inertia mass="${finger_mass}" x="${finger_length}" y="${finger_width}" z="${finger_height}"/>
+          <origin xyz="0 0 ${finger_length/2}" rpy = "0 0 0"/>
+        </inertial>
+      </link>
+        <!-- RIGHT FINGER -->
+        <link name="right_finger">
+            <visual>
+                <origin xyz="0 0 ${finger_length/2}" rpy="0 0 0"/>
+                <geometry>
+                    <box size="${finger_length} ${finger_width} ${finger_height}"/>
+                </geometry>
+                <material name="grey1"/>
+            </visual>
+            <collision>
+                <origin xyz="0 0 ${finger_length/2}" rpy="0 0 0"/>
+                <geometry>
+                    <box size="${finger_length} ${finger_width} ${finger_height}"/>
+                </geometry>
+            </collision>
+            <inertial>
+                <mass value="${finger_mass}"/>
+                <xacro:box_inertia mass="${finger_mass}" x="${finger_length}" y="${finger_width}" z="${finger_height}"/>
+                <origin xyz="0 0 ${finger_length/2}" rpy = "0 0 0"/>
+            </inertial>
+        </link>
+        <!-- JOINTS -->
+        <!-- Link 6 to Gripper -->
+        <joint name="gripper_base_joint" type="fixed">
+          <parent link="${parent}"/>
+          <child link="gripper_base"/>
+          <origin xyz="0 0 ${link6_length}" rpy="0 0 0"/>
+        </joint>
+        <!-- Left Finger to Gripper Base-->
+        <joint name="left_finger_joint" type="prismatic">
+          <parent link="gripper_base"/>
+          <child link="left_finger"/>
+          <origin xyz="0 ${gripper_base_width/2 +finger_height/2} ${gripper_base_height}" rpy="0 0 0"/>
+          <axis xyz="0 0 1"/>
+          <dynamics damping="0.5" friction="0.5"/>
+          <limit lower="0" upper="0.04"  effort="10" velocity="0.1"/>
+        </joint>
+        <!-- Right Finger to Gripper Base-->
+        <joint name="right_finger_joint" type="prismatic">
+          <parent link="gripper_base"/>
+          <child link="right_finger"/>
+          <origin xyz="0 ${-gripper_base_width/2 +finger_height/2} ${gripper_base_height}" rpy="0 0 0"/>
+          <axis xyz="0 0 1"/>
+          <dynamics damping="0.5" friction="0.5"/>
+          <limit lower="0" upper="0.04"  effort="10" velocity="0.1"/>
+        </joint>
+    </xacro:macro>
+</robot>

File: src/warehouse_robot_description/urdf/mobile_base.urdf.xacro (robot description, xacro)
@@ -11,126 +11,149 @@
     <xacro:property name="caster_radius" value="0.05"/>
     <xacro:property name="caster_mass" value="1.0"/>
-    <material name="blue">
-        <color rgba="0.2 0.2 0.8 1.0"/>
-    </material>
-    <material name="black">
-        <color rgba="0.1 0.1 0.1 1.0"/>
-    </material>
-    <material name="gray">
-        <color rgba="0.5 0.5 0.5 1.0"/>
-    </material>
-    <material name="white">
-        <color rgba="0.9 0.9 0.9 1.0"/>
-    </material>
+    <xacro:property name="mount_height" value="0.02"/>
+    <xacro:property name="mount_radius" value="0.12"/>
+    <xacro:property name="mount_mass" value="0.5"/>
     <!-- ============================== -->
     <!--          LINKS                 -->
     <!-- ============================== -->
     <!-- Base Link -->
-    <link name="base_link">
-        <visual>
+    <xacro:macro name="robot_base">
+        <link name="base_link">
+            <visual>
+                <origin xyz="0 0 0" rpy="0 0 0"/>
+                <geometry>
+                    <box size= "${base_length} ${base_width} ${base_height}"/>
+                </geometry>
+                <material name="grey1"/>
+            </visual>
+            <collision>
+                <origin xyz = "0 0 0" rpy = "0 0 0"/>
+                <geometry>
+                    <box size="${base_length} ${base_width} ${base_height}"/>
+                </geometry>
+            </collision>
+            <inertial>
+                <mass value="${base_mass}" />
+                <inertia ixx="0.1" iyy="0.33" izz="0.43"
+                        ixy="0.0" ixz="0.0" iyz="0.0"/>
+            </inertial>
+        </link>
+    <!-- Right Wheel -->
+        <link name="right_wheel">
+            <visual>
+                <origin xyz="0 0 0" rpy="1.57 0 0"/>
+                <geometry>
+                    <cylinder radius="${wheel_radius}" length="${wheel_length}"/>
+                </geometry>
+                <material name="black1"/>
+            </visual>
+            <collision>
+                <origin xyz="0 0 0" rpy="1.57 0 0"/>
+                <geometry>
+                    <cylinder radius="${wheel_radius}" length="${wheel_length}"/>
+                </geometry>
+            </collision>
+            <inertial>
+                <mass value="${wheel_mass}"/>
+                <inertia ixx="0.1" iyy="0.1" izz="0.1"
+                    ixy="0.0" ixz="0.0" iyz="0.0"/>
+            </inertial>
+        </link>
+        <!-- Left Wheel-->
+        <link name="left_wheel">
+            <visual>
+                <origin xyz="0 0 0" rpy="1.57 0 0"/>
+                <geometry>
+                    <cylinder radius="${wheel_radius}" length="${wheel_length}"/>
+                </geometry>
+                <material name="black1"/>
+            </visual>
+            <collision>
+                <origin xyz="0 0 0" rpy="1.57 0 0"/>
+                <geometry>
+                    <cylinder radius="${wheel_radius}" length="${wheel_length}"/>
+                </geometry>
+            </collision>
+            <inertial>
+                <mass value="${wheel_mass}"/>
+                <inertia ixx="0.1" iyy="0.1" izz="0.1"
+                    ixy="0.0" ixz="0.0" iyz="0.0"/>
+            </inertial>
+        </link>
+        <!-- Caster Wheel -->
+        <link name="caster_wheel">
+            <visual>
+                <origin xyz="0 0 0" rpy="1.57 0 0"/>
+                <geometry>
+                    <sphere radius="${caster_radius}"/>
+                </geometry>
+                <material name="white1"/>
+            </visual>
+            <collision>
+                <origin xyz="0 0 0" rpy="1.57 0 0"/>
+                <geometry>
+                    <sphere radius="${caster_radius}"/>
+                </geometry>
+            </collision>
+            <inertial>
+                <mass value="${caster_mass}"/>
+                <inertia ixx="0.1" iyy="0.1" izz="0.1"
+                    ixy="0.0" ixz="0.0" iyz="0.0"/>
+            </inertial>
+        </link>
+        <link name="mount_plate">
+            <visual>
+                <origin xyz="0 0 ${mount_height/2}" rpy="0 0 0"/>
+                <geometry>
+                    <cylinder radius="${mount_radius}" length="${mount_height}"/>
+                </geometry>
+                <material name="black1"/>
+            </visual>
+            <collision>
+                <origin xyz="0 0 ${mount_height/2}" rpy="0 0 0"/>
+                <geometry>
+                    <cylinder radius="${mount_radius}" length="${mount_height}"/>
+                </geometry>
+            </collision>
+            <inertial>
+                <mass value="${mount_mass}"/>
+                <inertia ixx="${mount_mass*(3*mount_radius*mount_radius + mount_height)/12}"
+                            iyy="${mount_mass*(3*mount_radius*mount_radius + mount_height)/12}"
+                            izz="${base_mass*(mount_radius*mount_radius)/2}"
+                            iyz="0.0"
+                            ixz="0.0"
+                            ixy="0.0"/>
+            </inertial>
+        </link>
+        <!-- ============================== -->
+        <!--          JOINTS                -->
+        <!-- ============================== -->
+        <!-- right to base wheel -->
+        <joint name="right_wheel_to_base" type="continuous">
+            <parent link="base_link"/>
+            <child link="right_wheel"/>
+            <origin xyz="0 -0.225 -${wheel_radius}" rpy="0 0 0"/>
+            <axis xyz="0 1 0"/>
+        </joint>
+        <!-- left wheel to base  -->
+        <joint name="left_wheel_to_base" type="continuous">
+            <parent link="base_link"/>
+            <child link="left_wheel"/>
+            <origin xyz="0 0.225 -${wheel_radius}" rpy="0 0 0"/>
+            <axis xyz="0 1 0"/>
+        </joint>
+        <!-- Caster Wheel to base-->
+        <joint name="caster_wheel_to_base" type="fixed">
+            <parent link="base_link"/>
+            <child link="caster_wheel"/>
+            <origin xyz="0.25 0 -0.15" rpy="0 0 0"/>
+            <axis xyz="0 1 0"/>
+        </joint>
+        <!-- Mount Link to Base -->
+        <joint name="mount_to_base" type="fixed">
+            <parent link="base_link"/>
+            <child link="mount_plate"/>
             <origin xyz="0 0 0" rpy="0 0 0"/>
-            <geometry>
-                <box size= "${base_length} ${base_width} ${base_height}"/>
-            </geometry>
-            <material name="blue"/>
-        </visual>
-        <collision>
-            <origin xyz = "0 0 0" rpy = "0 0 0"/>
-            <geometry>
-                <box size="${base_length} ${base_width} ${base_height}"/>
-            </geometry>
-        </collision>
-        <inertial>
-            <mass value="${base_mass}" />
-            <inertia ixx="0.1" iyy="0.33" izz="0.43"
-                    ixy="0.0" ixz="0.0" iyz="0.0"/>
-        </inertial>
-    </link>
-    <!-- Right Wheel -->
-    <link name="right_wheel">
-        <visual>
-            <origin xyz="0 0 0" rpy="1.57 0 0"/>
-            <geometry>
-                <cylinder radius="${wheel_radius}" length="${wheel_length}"/>
-            </geometry>
-            <material name="black"/>
-        </visual>
-        <collision>
-            <origin xyz="0 0 0" rpy="1.57 0 0"/>
-            <geometry>
-                <cylinder radius="${wheel_radius}" length="${wheel_length}"/>
-            </geometry>
-        </collision>
-        <inertial>
-            <mass value="${wheel_mass}"/>
-            <inertia ixx="0.1" iyy="0.1" izz="0.1"
-                ixy="0.0" ixz="0.0" iyz="0.0"/>
-        </inertial>
-    </link>
-    <!-- Left Wheel-->
-    <link name="left_wheel">
-        <visual>
-            <origin xyz="0 0 0" rpy="1.57 0 0"/>
-            <geometry>
-                <cylinder radius="${wheel_radius}" length="${wheel_length}"/>
-            </geometry>
-            <material name="black"/>
-        </visual>
-        <collision>
-            <origin xyz="0 0 0" rpy="1.57 0 0"/>
-            <geometry>
-                <cylinder radius="${wheel_radius}" length="${wheel_length}"/>
-            </geometry>
-        </collision>
-        <inertial>
-            <mass value="${wheel_mass}"/>
-            <inertia ixx="0.1" iyy="0.1" izz="0.1"
-                ixy="0.0" ixz="0.0" iyz="0.0"/>
-        </inertial>
-    </link>
-    <!-- Caster Wheel -->
-    <link name="caster_wheel">
-        <visual>
-            <origin xyz="0 0 0" rpy="1.57 0 0"/>
-            <geometry>
-                <sphere radius="${caster_radius}"/>
-            </geometry>
-            <material name="white"/>
-        </visual>
-        <collision>
-            <origin xyz="0 0 0" rpy="1.57 0 0"/>
-            <geometry>
-                <sphere radius="${caster_radius}"/>
-            </geometry>
-        </collision>
-        <inertial>
-            <mass value="${caster_mass}"/>
-            <inertia ixx="0.1" iyy="0.1" izz="0.1"
-                ixy="0.0" ixz="0.0" iyz="0.0"/>
-        </inertial>
-    </link>
-    <!-- ============================== -->
-    <!--          JOINTS                -->
-    <!-- ============================== -->
-    <!-- right to base wheel -->
-    <joint name="right_wheel_to_base" type="continuous">
-        <parent link="base_link"/>
-        <child link="right_wheel"/>
-        <origin xyz="0 -0.225 -${wheel_radius}" rpy="0 0 0"/>
-        <axis xyz="0 1 0"/>
-    </joint>
-    <!-- left wheel to base  -->
-    <joint name="left_wheel_to_base" type="continuous">
-        <parent link="base_link"/>
-        <child link="left_wheel"/>
-        <origin xyz="0 0.225 -${wheel_radius}" rpy="0 0 0"/>
-        <axis xyz="0 1 0"/>
-    </joint>
-    <!-- Caster Wheel to base-->
-    <joint name="caster_wheel_to_base" type="fixed">
-        <parent link="base_link"/>
-        <child link="caster_wheel"/>
-        <origin xyz="0.25 0 -0.15" rpy="0 0 0"/>
-        <axis xyz="0 1 0"/>
-    </joint>
+        </joint>
+    </xacro:macro>
 </robot>

File: src/warehouse_robot_description/urdf/robot.urdf.xacro (robot description, xacro)
@@ -1 +1,156 @@
-<
+<?xml version="1.0"?>
+<robot xmlns:xacro="http://www.ros.org/wiki/xacro" name="warehouse_mobile_manipulator">
+  <!-- ========================== -->
+  <!-- PROPERTIES -->
+  <!-- ========================== -->
+  <xacro:property name="my_pi" value="3.14159265359"/>
+    <!-- ========================== -->
+  <!-- MATERIALS -->
+  <!-- ========================== -->
+  <material name="blue1">
+      <color rgba="0.2 0.3 0.8 1.0"/>
+  </material>
+  <material name="orange1">
+      <color rgba="1.0 0.5 0.0 1.0"/>
+  </material>
+  <material name="red1">
+      <color rgba="0.8 0.2 0.2 1.0"/>
+  </material>
+  <material name="grey1">
+      <color rgba="0.6 0.6 0.6 1.0"/>
+  </material>
+  <material name="white1">
+      <color rgba="0.9 0.9 0.9 1.0"/>
+  </material>
+  <material name="black1">
+      <color rgba="0.1 0.1 0.1 1"/>
+  </material>
+  <!-- ========================== -->
+  <!-- INCLUDE MODULES -->
+  <!-- ========================== -->
+  <xacro:include filename="$(find warehouse_robot_description)/urdf/mobile_base.urdf.xacro"/>
+  <xacro:include filename="$(find warehouse_robot_description)/urdf/manipulator.urdf.xacro"/>
+  <xacro:include filename="$(find warehouse_robot_description)/urdf/gripper.urdf.xacro"/>
+  <xacro:include filename="$(find warehouse_robot_description)/urdf/sensors.urdf.xacro"/>
+  <!-- ========================== -->
+  <!-- INSTANTIATE MODULES -->
+  <!-- ========================== -->
+  <xacro:robot_base/>
+  <xacro:manipulator parent="mount_plate"/>
+  <xacro:gripper parent="link6"/>
+  <xacro:robot_sensors parent="base_link"/>
+  <!-- ========================== -->
+  <!-- GAZEBO MATERIALS -->
+  <!-- ========================== -->
+  <gazebo reference="main_base_link">
+    <material>Gazebo/Grey</material>
+    <mu1>0.2</mu1>
+    <mu2>0.2</mu2>
+  </gazebo>
+  <gazebo reference="right_wheel">
+    <material>Gazebo/Black</material>
+    <mu1>1.0</mu1>
+    <mu2>1.0</mu2>
+  </gazebo>
+  <gazebo reference="left_wheel">
+    <material>Gazebo/Black</material>
+    <mu1>1.0</mu1>
+    <mu2>1.0</mu2>
+  </gazebo>
+  <gazebo reference="caster_wheel">
+    <material>Gazebo/White</material>
+    <mu1>0.1</mu1>
+    <mu2>0.1</mu2>
+  </gazebo>
+  <!-- Arm links -->
+  <gazebo reference="link1"><material>Gazebo/Blue</material></gazebo>
+  <gazebo reference="link2"><material>Gazebo/Orange</material></gazebo>
+  <gazebo reference="link3"><material>Gazebo/Blue</material></gazebo>
+  <gazebo reference="link4"><material>Gazebo/Orange</material></gazebo>
+  <gazebo reference="link5"><material>Gazebo/Red</material></gazebo>
+  <gazebo reference="link6"><material>Gazebo/Blue</material></gazebo>
+  <!-- Gripper -->
+  <gazebo reference="gripper_base"><material>Gazebo/Grey</material></gazebo>
+  <gazebo reference="left_finger"><material>Gazebo/DarkGrey</material></gazebo>
+  <gazebo reference="right_finger"><material>Gazebo/DarkGrey</material></gazebo>
+  <!-- Sensors -->
+  <gazebo reference="lidar_link">
+    <material>Gazebo/Red</material>
+    <sensor type="ray" name="lidar_sensor">
+      <pose>0 0 0 0 0 0</pose>
+      <visualize>true</visualize>
+      <update_rate>10</update_rate>
+      <ray>
+        <scan>
+          <horizontal>
+            <samples>360</samples>
+            <resolution>1</resolution>
+            <min_angle>-3.14159</min_angle>
+            <max_angle>3.14159</max_angle>
+          </horizontal>
+        </scan>
+        <range>
+          <min>0.10</min>
+          <max>30.0</max>
+          <resolution>0.01</resolution>
+        </range>
+      </ray>
+      <plugin name="gazebo_ros_lidar" filename="libgazebo_ros_ray_sensor.so">
+        <ros>
+          <remapping>~/out:=scan</remapping>
+        </ros>
+        <output_type>sensor_msgs/LaserScan</output_type>
+      </plugin>
+    </sensor>
+  </gazebo>
+  <gazebo reference="camera_link">
+    <material>Gazebo/Black</material>
+    <sensor type="camera" name="camera_sensor">
+      <update_rate>30.0</update_rate>
+      <camera name="front_camera">
+        <horizontal_fov>1.3962634</horizontal_fov>
+        <image>
+          <width>640</width>
+          <height>480</height>
+          <format>R8G8B8</format>
+        </image>
+        <clip>
+          <near>0.02</near>
+          <far>300</far>
+        </clip>
+      </camera>
+      <plugin name="camera_controller" filename="libgazebo_ros_camera.so">
+        <ros>
+          <remapping>~/image_raw:=camera/image_raw</remapping>
+          <remapping>~/camera_info:=camera/camera_info</remapping>
+        </ros>
+        <camera_name>front_camera</camera_name>
+        <frame_name>camera_link</frame_name>
+      </plugin>
+    </sensor>
+  </gazebo>
+  <!-- ========================== -->
+  <!-- CONTROL PLUGINS -->
+  <!-- ========================== -->
+  <gazebo>
+    <plugin name="diff_drive_controller" filename="libgazebo_ros_diff_drive.so">
+      <ros>
+        <namespace>/</namespace>
+        <remapping>cmd_vel:=cmd_vel</remapping>
+        <remapping>odom:=odom</remapping>
+      </ros>
+      <update_rate>50</update_rate>
+      <left_joint>left_wheel_to_base</left_joint>
+      <right_joint>right_wheel_to_base</right_joint>
+      <wheel_separation>0.45</wheel_separation>
+      <wheel_diameter>0.2</wheel_diameter>
+      <max_wheel_torque>20</max_wheel_torque>
+      <max_wheel_acceleration>1.0</max_wheel_acceleration>
+      <publish_odom>true</publish_odom>
+      <publish_odom_tf>true</publish_odom_tf>
+      <publish_wheel_tf>true</publish_wheel_tf>
+      <odometry_frame>odom</odometry_frame>
+      <robot_base_frame>base_link</robot_base_frame>
+    </plugin>
+  </gazebo>
+</robot>
