Commit message: Warehouse robot Navigation

File: src/warehouse_robot_description/urdf/manipulator.urdf.xacro (robot description, xacro)
@@ -177,5 +177,5 @@
             <parent link="${parent}"/>
             <child link="link1"/>
-            <origin xyz="0 0 0" rpy="0 0 0"/>
+            <origin xyz="0 0 ${mount_height}" rpy="0 0 0"/>
             <axis xyz="0 0 1"/> <!-- Rotates around Z axis-->
             <dynamics damping="0.7" friction="0.5"/>

File: src/warehouse_robot_description/urdf/robot.urdf.xacro (robot description, xacro)
@@ -5,4 +5,5 @@
   <!-- ========================== -->
   <xacro:property name="my_pi" value="3.14159265359"/>
+  <xacro:property name="mount_height" value="0.02"/>
     <!-- ========================== -->
   <!-- MATERIALS -->
@@ -64,14 +65,66 @@
   </gazebo>
   <!-- Arm links -->
-  <gazebo reference="link1"><material>Gazebo/Blue</material></gazebo>
-  <gazebo reference="link2"><material>Gazebo/Orange</material></gazebo>
-  <gazebo reference="link3"><material>Gazebo/Blue</material></gazebo>
-  <gazebo reference="link4"><material>Gazebo/Orange</material></gazebo>
-  <gazebo reference="link5"><material>Gazebo/Red</material></gazebo>
-  <gazebo reference="link6"><material>Gazebo/Blue</material></gazebo>
+  <gazebo reference="link1">
+    <material>Gazebo/Blue</material>
+    <mu1>0.5</mu1>
+    <mu2>0.5</mu2>
+  </gazebo>
+  <gazebo reference="link2">
+    <material>Gazebo/Orange</material>
+    <mu1>0.5</mu1>
+    <mu2>0.5</mu2>
+  </gazebo>
+  <gazebo reference="link3">
+    <material>Gazebo/Blue</material>
+    <mu1>0.5</mu1>
+    <mu2>0.5</mu2>
+  </gazebo>
+  <gazebo reference="link4">
+    <material>Gazebo/Orange</material>
+    <mu1>0.5</mu1>
+    <mu2>0.5</mu2>
+  </gazebo>
+  <gazebo reference="link5">
+    <material>Gazebo/Red</material>
+    <mu1>0.5</mu1>
+    <mu2>0.5</mu2>
+  </gazebo>
+  <gazebo reference="link6">
+    <material>Gazebo/Blue</material>
+    <mu1>0.5</mu1>
+    <mu2>0.5</mu2>
+  </gazebo>
   <!-- Gripper -->
-  <gazebo reference="gripper_base"><material>Gazebo/Grey</material></gazebo>
-  <gazebo reference="left_finger"><material>Gazebo/DarkGrey</material></gazebo>
-  <gazebo reference="right_finger"><material>Gazebo/DarkGrey</material></gazebo>
+  <gazebo reference="gripper_base">
+    <material>Gazebo/Grey</material>
+    <mu1>0.5</mu1>
+    <mu2>0.5</mu2>
+  </gazebo>
+  <gazebo reference="left_finger">
+    <material>Gazebo/DarkGrey</material>
+    <mu1>1.2</mu1>
+    <mu2>1.2</mu2>
+  </gazebo>
+  <gazebo reference="right_finger">
+    <material>Gazebo/DarkGrey</material>
+    <mu1>1.2</mu1>
+    <mu2>1.2</mu2>
+  </gazebo>
+  <gazebo>
+    <plugin name="gazebo_ros_joint_state_publisher" filename="libgazebo_ros_joint_state_publisher.so">
+      <ros>
+        <remapping>~/out:=joint_states</remapping>
+      </ros>
+      <update_rate>50</update_rate>
+      <joint_name>joint1</joint_name>
+      <joint_name>joint2</joint_name>
+      <joint_name>joint3</joint_name>
+      <joint_name>joint4</joint_name>
+      <joint_name>joint5</joint_name>
+      <joint_name>joint6</joint_name>
+      <joint_name>left_finger_joint</joint_name>
+      <joint_name>right_finger_joint</joint_name>
+    </plugin>
+  </gazebo>
   <!-- Sensors -->
   <gazebo reference="lidar_link">
